File: moonratII/moonratII/moonratII.kicad_pcb (KiCad board)
At the start: 2 copper layers, 108 x 65 mm, 37 parts, among them J1 Barrel_Jack_Switch_SMT, J10 Conn_02x05_Odd_Even, J11 Screw_Terminal_01x02, J2 HS96L03W2C03_0.96_Oled, J3 PinHeader_1x06_P2.54mm_Vertic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, J4 PinHeader_1x08_P2.54mm_Vertic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, J5 Conn_02x05_Odd_Even, J6 Screw_Terminal_01x06, J7 PinHeader_1x08_P2.54mm_Vertic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, J8 PinHeader_1x10_P2.54mm_Vertic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, J9 Screw_Terminal_01x06, Q1 IRF520N, Q2 BSS138, SW1 6mm 2 Pin Tact NO Breadboard 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, SW2 6mm 2 Pin Tact NO Breadboard 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, SW3 6mm 2 Pin Tact NO Breadboard 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, U1 TMP36xS

Commit message: Add routing to the heater side.
Parts:
- J10, J5: footprint Connector_IDC:IDC-Header_2x06_P2.54mm_Vertical -> Connector_IDC:IDC-Header_2x05_P2.54mm_Vertical
- moved D1 13.0 mm to (151.1, 122.4)
- moved TP2 8.32 mm to (153.4, 146.3)
- moved U1 5.85 mm to (140.7, 121.9)
- moved R7 5.85 mm to (141.6, 128.4)
- moved J11 5.05 mm to (142.7, 136.1), turned to 0 degrees
- moved J10 2.18 mm to (149.1, 107.5)
- moved H5 2.00 mm to (144.0, 89.0)
- moved H6 2.00 mm to (144.0, 146.0)
- moved J9 0.35 mm to (151.0, 98.0)
Routing:
- net GND: track 341.3 -> 0.00 mm
- net VCC: track 101.8 -> 0.00 mm
- net +5V: track 80.2 -> 0.00 mm
- net BTN_DOWN: track 74.3 -> 0.00 mm
- net GND1: track 54.9 -> 0.00 mm, vias 0 -> 12
- net VCCQ: track 20.7 -> 69.5 mm, vias 0 -> 3
- net BTN_UP: track 41.3 -> 0.00 mm
- net (no net): track 39.8 -> 0.00 mm
- net BTN_SELECT: track 34.1 -> 0.00 mm
- net TempOut: track 24.2 -> 0.00 mm
- net HeaterDrive_IB: track 20.3 -> 43.0 mm, vias 0 -> 1
- net HeaterDrive: track 17.4 -> 0.00 mm
- net +5P: track 31.6 -> 46.1 mm, vias 0 -> 1
- net TempOut_IB: track 28.9 -> 40.0 mm, vias 0 -> 1
- net TEMP_IN: track 10.5 -> 0.00 mm
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- added copper zone on B.Cu, net GND1
- added copper zone on F.Cu, net GND1
