File: moonratII/moonratII/moonratII.kicad_sch (KiCad schematic)
At the start: 40 parts, among them J1 Barrel_Jack_Switch_SMT, J10 Conn_02x05_Odd_Even, J11 Screw_Terminal_01x02, J2 HS96L03W2C03_0.96_Oled, J3 Conn_01x06_Male, J4 Conn_01x08_Male, J5 Conn_02x05_Odd_Even, J6 Screw_Terminal_01x06, J7 Conn_01x08_Male, J8 Conn_01x10_Male, J9 Screw_Terminal_01x06, Q1 IRF520N, Q2 BSS138, SW1 6mm 2 Pin Tact NO Breadboard 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, SW2 6mm 2 Pin Tact NO Breadboard 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, SW3 6mm 2 Pin Tact NO Breadboard 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, U1 TMP36xS

Commit message: Add routing to the heater side.
Parts:
- J10, J5: footprint Connector_IDC:IDC-Header_2x06_P2.54mm_Vertical -> Connector_IDC:IDC-Header_2x05_P2.54mm_Vertical
Changed lines of the file:
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@@
       (effects (font (size 1.27 1.27)))
     )
-    (property "Footprint" "Connector_IDC:IDC-Header_2x06_P2.54mm_Vertical" (at 204.47 153.67 0)
+    (property "Footprint" "Connector_IDC:IDC-Header_2x05_P2.54mm_Vertical" (at 204.47 153.67 0)
       (effects (font (size 1.27 1.27)) hide)
     )
@@
       (effects (font (size 1.27 1.27)))
     )
-    (property "Footprint" "Connector_IDC:IDC-Header_2x06_P2.54mm_Vertical" (at 148.59 153.67 0)
-      (effects (font (size 1.27 1.27)) hide)
-    )
+    (property "Footprint" "Connector_IDC:IDC-Header_2x05_P2.54mm_Vertical" (at 148.59 153.67 0)
+      (effects (font (size 1.27 1.27)) hide)
+    )
